File: pcb/smart-doorbell/smart-doorbell.kicad_sch (KiCad schematic)
At the start: 53 parts, among them J1 Conn_01x02_Pin, J2 USB_C_Receptacle_USB2.0_16P, J3 Conn_01x24, J4 Conn_01x06, J6 Conn_01x02_Pin, J7 Conn_01x03, J8 Conn_01x04, U1 ESP32-S3-WROOM-2, U2 MCP73831-2-OT, U3 AP2112K-3.3, U4 MAX98357A, U5 SRV05-4, U6 XC6206P152MR, U7 XC6206P282MR

Commit message: Update Rev B camera hardware outputs
Parts:
- removed U1: ESP32-S3-WROOM-2, RF_Module:ESP32-S3-WROOM-2, symbol RF_Module:ESP32-S3-WROOM-2
- added R15: 680, Resistor_SMD:R_0603_1608Metric, symbol Device:R_US
- added R16: 3.9k, Resistor_SMD:R_0603_1608Metric, symbol Device:R_US
- added R17, R19: 10k, Resistor_SMD:R_0603_1608Metric, symbol Device:R_US
- added R18, R20: 56k, Resistor_SMD:R_0603_1608Metric, symbol Device:R_US
- added U1: ESP32-S3-WROOM-1, RF_Module:ESP32-S3-WROOM-1, symbol RF_Module:ESP32-S3-WROOM-1
Connections:
- net +2V8: now also C22.2, J3.11 (Pin_11), R13.2, R14.2
- net +3V3: now also U1.2 (3V3); no longer C22.2, J3.11 (Pin_11), R13.2, R14.2
- net AMP_EN: now also U1.36 (RXD0)
- net BTN_LED: now also U1.25 (IO48)
- net CAM_D0: now also U1.11 (IO18)
- net CAM_D1: now also U1.9 (IO16)
- net CAM_D2: now also U1.8 (IO15)
- net CAM_D3: now also U1.10 (IO17)
- net CAM_D4: now also U1.12 (IO8)
- net CAM_D5: now also U1.18 (IO10)
- net CAM_D6: now also U1.19 (IO11)
- net CAM_D7: now also U1.21 (IO13)
- net CAM_HREF: now also U1.22 (IO14)
- net CAM_PCLK: now also U1.17 (IO9)
- net CAM_PWDN: now also R19.1, U1.23 (IO21); no longer J3.8 (Pin_8)
- net CAM_RST: now also R17.1, U1.33 (IO40); no longer J3.6 (Pin_6)
- net CAM_SCL: now also U1.32 (IO39)
- net CAM_SDA: now also U1.31 (IO38)
- net CAM_VSYNC: now also U1.34 (IO41)
- net CAM_XCLK: now also R15.1, U1.20 (IO12); no longer J3.13 (Pin_13)
- net DOORBELL_IN: now also U1.38 (IO2)
- net GND: now also R16.2, R18.2, R20.2, U1.1 (GND), U1.40 (GND), U1.41 (GND)
- net GPIO1: now also U1.39 (IO1)
- net GPIO19: now also U1.13 (USB_D-)
- net GPIO20: now also U1.14 (USB_D+)
- net GPIO4: now also U1.4 (IO4)
- net GPIO5: now also U1.5 (IO5)
- net GPIO6: now also U1.6 (IO6)
- net GPIO7: now also U1.7 (IO7)
- net PIR_OUT: now also U1.35 (IO42)
- net STATUS_LED: now also U1.24 (IO47)
- net at C14.2, R1.2, RESET1.2 (B): now also U1.3 (EN)
- net at BOOT1.1 (A): now also U1.27 (IO0)
- new net CAM_PWDN_2V8: J3.8 (Pin_8), R19.2, R20.1
- new net CAM_RST_2V8: J3.6 (Pin_6), R17.2, R18.1
- new net CAM_XCLK_2V8: J3.13 (Pin_13), R15.2, R16.1
- no-connect marks 9 -> 12
Other:
- note added: "ESP32-S3-WROOM-1"
- note removed: "ESP32-S3-WROOM-2"
- moved on the sheet: BOOT1, C1, C14, C2, C20, C21, C22, C23, C25, C3, C9, D3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

Commit message: Release Smart Doorbell Rev B PCB order snapshot
Record the exact JLCPCB Gerber, BOM, and CPL files submitted on 2026-07-15, including project-local part/placement corrections and the verified native top-mask repair. Preserve the routed KiCad sources, production netlists, custom power footprints, camera documentation, assembly exclusions, and release hashes used for the five-board first-article order.
Parts:
- removed U2: MCP73831-2-OT, Package_TO_SOT_SMD:SOT-23-5, symbol Battery_Management:MCP73831-2-OT
- removed U3: AP2112K-3.3, Package_TO_SOT_SMD:SOT-23-5, symbol Regulator_Linear:AP2112K-3.3
- added C11, C28, C30: 0.1u, Capacitor_SMD:C_0603_1608Metric, symbol Device:C
- added C24, C29, C31: 22u, Capacitor_SMD:C_0603_1608Metric, symbol Device:C
- added C32, C33, C34: 10u, Capacitor_SMD:C_0603_1608Metric, symbol Device:C
- added H1, H2, H3, H4: MountingHole_2.7mm_M2.5, MountingHole:MountingHole_2.7mm_M2.5, symbol Mechanical:MountingHole
- added J5: NTC_OPTION, Connector_Wire:SolderWire-0.25sqmm_1x02_P4.2mm_D0.65mm_OD1.7mm, symbol Connector_Generic:Conn_01x02
- added J9: Conn_01x04, Connector_PinHeader_2.54mm:PinHeader_1x04_P2.54mm_Vertical, symbol Connector_Generic:Conn_01x04
- added L1: 0.47u, Inductor_SMD:L_1008_2520Metric, symbol Device:L
- added R11, R21, R32, R36: 0, Resistor_SMD:R_0603_1608Metric, symbol Device:R_US
- added R22: 511k, Resistor_SMD:R_0603_1608Metric, symbol Device:R_US
- added R23: 91k, Resistor_SMD:R_0603_1608Metric, symbol Device:R_US
- added R24, R29, R38: 100k, Resistor_SMD:R_0603_1608Metric, symbol Device:R_US
- added R25: 25k, Resistor_SMD:R_0603_1608Metric, symbol Device:R_US
- added R26, R33: 10k, Resistor_SMD:R_0603_1608Metric, symbol Device:R_US
- added R27: 330k, Resistor_SMD:R_0603_1608Metric, symbol Device:R_US
- added R28: 110k, Resistor_SMD:R_0603_1608Metric, symbol Device:R_US
- added R30, R31, R37, R39, R40: 1k, Resistor_SMD:R_0603_1608Metric, symbol Device:R_US
- added R34, R35: 22, Resistor_SMD:R_0603_1608Metric, symbol Device:R_US
- added TP1, TP10, TP2, TP3, TP4, TP5, TP6, TP7, TP8, TP9: TestPoint, TestPoint:TestPoint_Pad_D1.0mm, symbol Connector:TestPoint
- added U2: MCP73871T-2AAI/ML, Package_DFN_QFN:QFN-20-1EP_4x4mm_P0.5mm_EP2.5x2.5mm, symbol Battery_Management:MCP73871-2CC
- added U8: TPS63802DLAR, smart-doorbell-power:TPS63802DLAR_DLA0010A, symbol smart-doorbell-power:TPS63802DLAR
- added U9: TPS22919DCK, Package_TO_SOT_SMD:SOT-363_SC-70-6, symbol Power_Management:TPS22919DCK
- BOOT1, RESET1: LCSC Part # (none) -> C231329
- C1, C13, C20, C25, C26, C3: LCSC Part # (none) -> C19702
- C27: value 10u -> 22u; LCSC Part # (none) -> C84419
- J1, J6: LCSC Part # (none) -> C131337
- J2: LCSC Part # (none) -> C165948
- J3: LCSC Part # (none) -> C202112
- J4: LCSC Part # (none) -> C37208
- J7: LCSC Part # (none) -> C131339
- J8: LCSC Part # (none) -> C131334
- MK1, U1: now left out of the parts list
- R1, R17, R19, R5: LCSC Part # (none) -> C15401
- R12: value 2k -> 4.7k
- R3: LCSC Part # (none) -> C21190
- R4, R7, R8: LCSC Part # (none) -> C25803
- U4: footprint Package_DFN_QFN:TQFN-16-1EP_3x3mm_P0.5mm_EP1.23x1.23mm -> smart-doorbell-power:MAX98357A_TQFN-16-1EP_3x3mm_P0.5mm_EP1.23x1.23mm
- U6: value XC6206P152MR -> DS8561-15S3; LCSC Part # (none) -> C5795628; MPN (none) -> DS8561-15S3
Connections:
- net +1V5: now also TP8.1
- net +2V8: now also R11.2, TP7.1; no longer J3.24 (Pin_24)
- net +3V3: now also C29.1, C30.1, R22.2, R33.1, R36.1, TP6.1, U8.6 (VOUT), U9.1 (IN); no longer C15.1, C17.1, U6.3 (VI), U7.3 (VI)
- net +5V: now also C24.1, R27.1, TP3.1, U2.17 (CE), U2.18 (IN), U2.19 (IN), U2.4 (PROG2)
- net +BATT: now also C33.2, C34.2, TP4.1, U2.14 (V_{BAT}), U2.15 (V_{BAT}), U2.16 (V_{BAT_SENSE}); no longer C26.1, U4.7 (VDD), U4.8 (VDD)
- net GND: now also C11.1, C24.2, C28.2, C29.2, C30.2, C31.2, C32.2, C33.1, C34.1, J5.2 (Pin_2), J9.2 (Pin_2), R21.2, R23.2, R25.1, R26.1, R28.1, R29.1, R38.1, TP9.1, U2.10 (V_{SS}), U2.11 (V_{SS}), U2.21 (V_{SS}), U2.3 (SEL), U2.9 (~{TE}), U8.2 (MODE), U8.3 (AGND), U8.8 (GND), U9.2 (GND); no longer J3.23 (Pin_23)
- net GPIO19: now also R35.2; no longer J2.A7 (D-), J2.B7 (D-), U5.4 (IO3)
- net GPIO20: now also R34.2; no longer J2.A6 (D+), J2.B6 (D+), U5.3 (IO2)
- net PIR_WAKE: now reaches U1.15 (IO3)
- net PIR_WAKE: now also R30.2
- net at BOOT1.1 (A), U1.27 (IO0): now also R33.2
- net GPIO43_AUX: now reaches U1.37 (TXD0)
- net GPIO43_AUX: now also R40.1
- net at R12.2: now also U2.13 (PROG1)
- net at D2.1 (K): now also U2.8 (STAT1/~{LBO})
- net at U4.2 (GAIN_SLOT): now also R32.1
- net PIR_OUT renamed GPIO42_AUX
- net GPIO42_AUX: now also R31.2, R37.1, R39.1; no longer J7.2 (Pin_2)
- new net: J9.3 (Pin_3), R39.2
- new net: J3.24 (Pin_24), R11.1, TP1.1
- new net: R25.2, U2.12 (PROG3)
- new net: J3.23 (Pin_23), R21.1, TP2.1
- new net: L1.1, U8.7 (L2)
- new net: L1.2, U8.9 (L1)
- new net: R24.2, U8.1 (EN)
- new net: R22.1, R23.1, U8.4 (FB)
- new net: J9.4 (Pin_4), R40.2
- new net: R27.2, R28.2, U2.2 (VPCC)
- new net BATT_THERM: J5.1 (Pin_1), R26.2, U2.5 (THERM)
- new net CAM_3V3: C15.1, C17.1, R36.2, TP10.1, U6.3 (VI), U7.3 (VI), U9.6 (OUT)
- new net CAM_PWR_EN: R37.2, R38.2, U9.3 (ON)
- new net PIR_SENSOR_OUT: J7.2 (Pin_2), R29.2, R30.1, R31.1
- new net SYS: C11.2, C26.1, C28.1, C31.1, C32.1, J9.1 (Pin_1), R24.1, R32.2, TP5.1, U2.1 (OUT), U2.20 (OUT), U4.7 (VDD), U4.8 (VDD), U8.10 (VIN)
- new net U5_IO2: J2.A6 (D+), J2.B6 (D+), R34.1, U5.3 (IO2)
- new net U5_IO3: J2.A7 (D-), J2.B7 (D-), R35.1, U5.4 (IO3)
- no-connect marks 12 -> 13
Other:
- note added: "OPTIONAL BATTERY NTC"
- moved on the sheet: BOOT1, C13, C26, C27, D2, J7, R12, R15, R16, R17, R18, R19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

Commit message: Prepare Smart Doorbell Rev C reorder
Correct and verify the mirrored OV5640 interface, add switched camera power control and hardware bring-up modes, preserve the ordered Rev B artifacts, and add an isolated integrity-locked Rev C JLCPCB release candidate with updated documentation.
Parts:
- added C35: 1u, Capacitor_SMD:C_0603_1608Metric, symbol Device:C
- J3: symbol Connector_Generic:Conn_01x24 -> ov5640_pinout:OV5640_FPC_24
- R26, R36: now not fitted
- R37: now fitted
- U9: LCSC Part # (none) -> C2149796; now fitted
Connections:
- net +1V5: now also J3.15 (CAM10_DVDD); no longer J3.10 (Pin_10)
- net +2V8: now also J3.14 (CAM11_DOVDD), J3.21 (CAM4_AVDD); no longer J3.11 (Pin_11), J3.4 (Pin_4)
- net +3V3: now also C35.2
- net CAM_D0: now also J3.6 (CAM19_Y2_D0); no longer J3.19 (Pin_19)
- net CAM_D1: now also J3.4 (CAM21_Y3_D1); no longer J3.21 (Pin_21)
- net CAM_D2: now also J3.3 (CAM22_Y4_D2); no longer J3.22 (Pin_22)
- net CAM_D3: now also J3.5 (CAM20_Y5_D3); no longer J3.20 (Pin_20)
- net CAM_D4: now also J3.7 (CAM18_Y6_D4); no longer J3.18 (Pin_18)
- net CAM_D5: now also J3.9 (CAM16_Y7_D5); no longer J3.16 (Pin_16)
- net CAM_D6: now also J3.11 (CAM14_Y8_D6); no longer J3.14 (Pin_14)
- net CAM_D7: now also J3.13 (CAM12_Y9_D7); no longer J3.12 (Pin_12)
- net CAM_HREF: now also J3.16 (CAM9_HREF); no longer J3.9 (Pin_9)
- net CAM_PCLK: now also J3.8 (CAM17_PCLK); no longer J3.17 (Pin_17)
- net CAM_PWDN_2V8: now also J3.17 (CAM8_PWDN); no longer J3.8 (Pin_8)
- net CAM_RST_2V8: now also J3.19 (CAM6_RESET); no longer J3.6 (Pin_6)
- net CAM_SCL: now also J3.20 (CAM5_SIO_C); no longer J3.5 (Pin_5)
- net CAM_SDA: now also J3.22 (CAM3_SIO_D); no longer J3.3 (Pin_3)
- net CAM_VSYNC: now also J3.18 (CAM7_VSYNC); no longer J3.7 (Pin_7)
- net CAM_XCLK_2V8: now also J3.12 (CAM13_XCLK); no longer J3.13 (Pin_13)
- net GND: now also J3.10 (CAM15_DGND), J3.23 (CAM2_AGND), C35.1; no longer J3.15 (Pin_15), J3.2 (Pin_2)
- net at R11.1, TP1.1: now also J3.1 (CAM24_AFVDD); no longer J3.24 (Pin_24)
- net at R21.1, TP2.1: now also J3.2 (CAM23_AF_GND); no longer J3.23 (Pin_23)
Other:
- title: (none) -> Smart Doorbell Project
- moved on the sheet: R11, R13, R14, R21, TP1, TP2, TP9
