File: pcb/smart-doorbell/smart-doorbell.kicad_pcb (KiCad board)
At the start: 2 copper layers, 59 x 91 mm, 107 parts, among them J1 Conn_01x02_Pin, J2 USB_C_Receptacle_USB2.0_16P, J3 Conn_01x24, J4 Conn_01x06, J5 NTC_OPTION, J6 Conn_01x02_Pin, J7 Conn_01x03, J8 Conn_01x04, J9 Conn_01x04, U1 ESP32-S3-WROOM-1, U2 MCP73871T-2AAI/ML, U4 MAX98357A, U5 SRV05-4, U6 DS8561-15S3, U7 XC6206P282MR, U8 TPS63802DLAR, U9 TPS22919DCK

Commit message: Prepare Smart Doorbell Rev C reorder
Correct and verify the mirrored OV5640 interface, add switched camera power control and hardware bring-up modes, preserve the ordered Rev B artifacts, and add an isolated integrity-locked Rev C JLCPCB release candidate with updated documentation.
Parts:
- added C35: 1u, Capacitor_SMD:C_0603_1608Metric, F.Cu at (124.8, 110.3)
- moved TP1 21.4 mm to (148.0, 100.0)
- moved R21 17.4 mm to (145.1, 98.3), turned to -90 degrees
- moved R11 15.8 mm to (143.5, 98.3), turned to -90 degrees
- moved TP2 15.8 mm to (144.7, 101.2)
- moved R36 6.65 mm to (126.4, 106.5)
- moved TP7 6.21 mm to (140.0, 110.8)
- moved H3 6.00 mm to (111.0, 128.8)
- moved H4 6.00 mm to (162.4, 128.8)
- moved TP10 3.93 mm to (126.4, 103.5)
- moved U9 3.54 mm to (126.8, 113.0)
- moved D2 1.90 mm to (149.9, 140.7)
- moved C15 1.77 mm to (129.9, 107.8)
- moved U6 1.65 mm to (131.8, 105.8)
- moved TP8 1.25 mm to (133.8, 109.5)
- moved C25 1.12 mm to (130.6, 98.4)
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Connections:
- J3 pad 1: unconnected-(J3-Pin_1-Pad1) -> Net-(J3-CAM24_AFVDD)
- J3 pad 10: +1V5 -> GND
- J3 pad 11: +2V8 -> /CAM_D6
- J3 pad 12: /CAM_D7 -> /CAM_XCLK_2V8
- J3 pad 13: /CAM_XCLK_2V8 -> /CAM_D7
- J3 pad 14: /CAM_D6 -> +2V8
- J3 pad 15: GND -> +1V5
- J3 pad 16: /CAM_D5 -> /CAM_HREF
- J3 pad 17: /CAM_PCLK -> /CAM_PWDN_2V8
- J3 pad 18: /CAM_D4 -> /CAM_VSYNC
- J3 pad 19: /CAM_D0 -> /CAM_RST_2V8
- J3 pad 2: GND -> Net-(J3-CAM23_AF_GND)
- J3 pad 20: /CAM_D3 -> /CAM_SCL
- J3 pad 21: /CAM_D1 -> +2V8
- J3 pad 22: /CAM_D2 -> /CAM_SDA
- J3 pad 23: Net-(J3-Pin_23) -> GND
- J3 pad 24: Net-(J3-Pin_24) -> unconnected-(J3-CAM1_NC-Pad24)
- J3 pad 3: /CAM_SDA -> /CAM_D2
- J3 pad 4: +2V8 -> /CAM_D1
- J3 pad 5: /CAM_SCL -> /CAM_D3
- J3 pad 6: /CAM_RST_2V8 -> /CAM_D0
- J3 pad 7: /CAM_VSYNC -> /CAM_D4
- J3 pad 8: /CAM_PWDN_2V8 -> /CAM_PCLK
- J3 pad 9: /CAM_HREF -> /CAM_D5
- R11 pad 1: Net-(J3-Pin_24) -> Net-(J3-CAM24_AFVDD)
- R21 pad 1: Net-(J3-Pin_23) -> Net-(J3-CAM23_AF_GND)
- TP1 pad 1: Net-(J3-Pin_24) -> Net-(J3-CAM24_AFVDD)
- TP2 pad 1: Net-(J3-Pin_23) -> Net-(J3-CAM23_AF_GND)
Routing:
- net GND: track 529.4 -> 541.5 mm
- net Net-(J3-Pin_24): track 12.0 -> 0.00 mm
- net Net-(J3-Pin_23): track 11.5 -> 0.00 mm
- net +2V8: track 89.8 -> 101.1 mm, vias 4 -> 6
- net /CAM_XCLK_2V8: track 24.2 -> 13.5 mm
- net Net-(J3-CAM24_AFVDD): track 0.00 -> 10.6 mm
- net /CAM_XCLK: track 19.5 -> 29.5 mm
- net Net-(J3-CAM23_AF_GND): track 0.00 -> 9.83 mm, vias 0 -> 4
- net /CAM_SDA: track 46.0 -> 54.7 mm, vias 6 -> 4
- net /SYS: track 171.1 -> 178.7 mm
- net /CAM_RST: track 34.0 -> 26.6 mm
- net /CAM_HREF: track 12.7 -> 19.2 mm, vias 0 -> 2
- net /CAM_PWDN_2V8: track 16.9 -> 11.9 mm
- net /CAM_VSYNC: track 27.7 -> 32.0 mm
- net /CAM_D4: track 22.1 -> 25.9 mm
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Other:
- outline, holes or cut-outs redrawn
- board text added: "CAM1/ J3-24"
- board text added: "CAM24/ J3-1"
- board text added: "FLEX ENTRY"
- board text added: "MIC PORT DO NOT COVER"
- board text added: "Smart Doorbell Project Rev C"
- board text removed: "Smart Doorbell Project Rev B"

Commit message: Record ordered Smart Doorbell Rev C release
Freeze the exact five-board JLCPCB upload package, order identifiers, BOM matching export, and signed-off assembly preview. Preserve the immutable Rev B release, record the locked PCB state and regenerated manufacturing files, and document the selected 10 mm enclosure standoffs.
Other:
- board text added: "CAM1 / J3-24"
- board text added: "CAM24 / J3-1"
- board text removed: "CAM1/ J3-24"
- board text removed: "CAM24/ J3-1"
